Commit message: changed to work with Franka NBV

File: pb_ros/src/pb_ros/urdf/urdf/ur5.xacro (robot description, xacro)
@@ -1,3 +1,3 @@
-<?xml version="1.0" ?>
+<?xml version="1.0" encoding='utf-8'?>
 <!-- =================================================================================== -->
 <!-- |    This document was autogenerated by xacro from sisbot.xacro                   | -->
@@ -5,8 +5,22 @@
 <!-- =================================================================================== -->
 <robot name="sisbot" xmlns:xacro="http://ros.org/wiki/xacro">
-<!-- <robot name="sisbot" xmlns:xacro="http://ros.org/wiki/xacro"> -->
   <!--################################################
   ########              arm                    #######
   ####################################################-->
+<xacro:macro name="ur5_arm" params="connected_to:='' ns:='panda' xyz:='0 0 0' rpy:='0 0 0' safety_distance:=0">
+  <!-- connect arm to panda world -->
+  <xacro:unless value="${not connected_to}">
+    <!-- <joint name="${connected_to}_ur5_joint" type="fixed"> -->
+    <joint name="panda_ur5_joint" type="fixed">
+      <parent link="${connected_to}"/>
+      <child link="base_link"/>
+      <origin rpy="${rpy}" xyz="${xyz}"/>
+    </joint>
+    <!-- <joint name="${connected_to}_ur5_floating_joint1" type="floating">
+      <parent link="${connected_to}"/>
+      <child link="shoulder_link"/>
+      <origin rpy="${rpy}" xyz="${xyz}"/>
+    </joint> -->
+  </xacro:unless>
   <link name="base_link">
     <visual>
@@ -197,4 +211,12 @@
     </inertial>
   </link>
+  <link name="ee_link">
+    <collision>
+      <geometry>
+        <box size="0.01 0.01 0.01"/>
+      </geometry>
+      <origin rpy="0 0 0" xyz="-0.01 0 0"/>
+    </collision>
+  </link>
   <joint name="ee_fixed_joint" type="fixed">
     <parent link="wrist_3_link"/>
@@ -202,13 +224,5 @@
     <origin rpy="0.0 0.0 1.57079632679" xyz="0.0 0.0823 0.0"/>
   </joint>
-  <link name="ee_link">
-    <collision>
-      <geometry>
-        <box size="0.01 0.01 0.01"/>
-      </geometry>
-      <origin rpy="0 0 0" xyz="-0.01 0 0"/>
-    </collision>
-  </link>
-  <link name="camera_depth_optical_frame">
+  <link name="ur5_camera_depth_optical_frame">
     <inertial>
       <origin rpy="0 0 0" xyz="0 0 0"/>
@@ -220,5 +234,5 @@
     <!-- <parent link="panda_hand"/> -->
     <parent link="ee_link"/>
-    <child link="camera_depth_optical_frame"/>
+    <child link="ur5_camera_depth_optical_frame"/>
     <!-- original working-->
     <!-- <origin rpy="0 0 1.570" xyz="0.06 0 0.02"/> -->
@@ -229,11 +243,11 @@
   ########          connect model                #####
   ####################################################-->
-  <!-- connect arm to world -->
-  <link name="world"/>
+  <!-- <link name="world"/> -->
   <!-- <link name="panda_link0" /> -->
-  <joint name="world_joint" type="fixed">
+  <!-- <joint name="world_joint" type="fixed">
     <parent link="world"/>
     <child link="base_link"/>
     <origin rpy="0.0 0.0 0" xyz="0.0 0.0 2.1"/>
-  </joint>
+  </joint> -->
+  </xacro:macro>
 </robot>
