Commit message: ur5 sim working, nbv control not working

File: pb_ros/src/pb_ros/urdf/urdf/ur5.urdf (robot description, URDF)
Before this commit: robot sisbot, 10 links, 9 joints
Links:
- removed link camera_depth_optical_frame
- added link ur5_camera_depth_optical_frame, mass 0.0
Joints:
- removed joint world_joint
- added joint world_ur5_joint: type fixed, parent world, child base_link, origin xyz=0.0 0.0 0 rpy=0.0 0.0 0
- joint ur5_hand_camera_depth_optical_frame_joint: child camera_depth_optical_frame -> ur5_camera_depth_optical_frame; origin xyz=0 0.0 0.05 rpy=0 0 0 -> xyz=0.0 0.0 -0.05 rpy=1.570 0 1.57

File: pb_ros/src/pb_ros/urdf/urdf/ur5.xacro (robot description, xacro)
@@ -11,6 +11,6 @@
   <!-- connect arm to panda world -->
   <xacro:unless value="${not connected_to}">
-    <!-- <joint name="${connected_to}_ur5_joint" type="fixed"> -->
-    <joint name="panda_ur5_joint" type="fixed">
+    <joint name="${connected_to}_ur5_joint" type="fixed">
+    <!-- <joint name="panda_ur5_joint" type="fixed"> -->
       <parent link="${connected_to}"/>
       <child link="base_link"/>
@@ -238,16 +238,7 @@
     <!-- <origin rpy="0 0 1.570" xyz="0.06 0 0.02"/> -->
     <!-- mine -->
-    <origin rpy="0 0 0" xyz="0 0.0 0.05"/>
-  </joint>
-  <!--################################################
-  ########          connect model                #####
-  ####################################################-->
-  <!-- <link name="world"/> -->
-  <!-- <link name="panda_link0" /> -->
-  <!-- <joint name="world_joint" type="fixed">
-    <parent link="world"/>
-    <child link="base_link"/>
-    <origin rpy="0.0 0.0 0" xyz="0.0 0.0 2.1"/>
-  </joint> -->
+    <!-- <origin rpy="0 0 0" xyz="0 0.0 0.05"/> -->
+    <origin rpy="1.570 0 1.57" xyz="0 0.0 -0.05"/>
+  </joint>
   </xacro:macro>
 </robot>
